File: documents/cwater/cwater.kicad_pcb (KiCad board)
At the start: 2 copper layers, 66.2 x 89.1 mm, 40 parts, among them IC10 MAX635, IC11 LP324N, IC7 MAX603, J1 Conn_01x12, J2 Conn_01x08, J3 Conn_02x08_Top_Bottom, J4 Conn_02x06_Top_Bottom, J5 Conn_02x10_Top_Bottom, J6 Conn_02x08_Top_Bottom, U1 AT45DB161D-SU

Commit message: prepare for reinstallation
Other:
- net class Default removed
